File: sensus-breakout.kicad_sch (KiCad schematic)
At the start: 7 parts, among them J1 v1 connector, J2 Breakout, J3 JLink, J5 USB_B_Micro, U1 XC6206P332MR

Commit message: Ordered second version of breakout board.
Parts:
- removed J2: Breakout, Connector_PinHeader_2.54mm:PinHeader_1x10_P2.54mm_Vertical, symbol Connector_Generic:Conn_01x10
- removed J3: JLink, Connector_PinHeader_1.27mm:PinHeader_2x05_P1.27mm_Vertical_SMD, symbol Connector_Generic:Conn_02x05_Odd_Even
- added C10, C11: 1u, Capacitor_SMD:C_0402_1005Metric, symbol Device:C_Small
- added C12, C3, C6, C7, C8, C9: 100n, Capacitor_SMD:C_0402_1005Metric, symbol Device:C_Small
- added C4, C5: 30p, Capacitor_SMD:C_0402_1005Metric, symbol Device:C_Small
- added D1: LED_Small, LED_SMD:LED_0603_1608Metric, symbol Device:LED_Small
- added J2: USB_BOOT, Connector_PinHeader_2.54mm:PinHeader_1x02_P2.54mm_Vertical, symbol Connector_Generic:Conn_01x02
- added J3: Conn_01x08, Connector_PinHeader_2.54mm:PinHeader_1x08_P2.54mm_Vertical, symbol Connector_Generic:Conn_01x08
- added R1, R2: 27, Resistor_SMD:R_0603_1608Metric, symbol Device:R_Small
- added R3, R7: 1k, Resistor_SMD:R_0402_1005Metric, symbol Device:R_Small
- added R4: 10k, Resistor_SMD:R_0402_1005Metric, symbol Device:R_Small
- added R5, R6: 100, Resistor_SMD:R_0402_1005Metric, symbol Device:R_Small
- added U2: RP2040, Package_DFN_QFN:QFN-56-1EP_7x7mm_P0.4mm_EP3.2x3.2mm, symbol MCU_RaspberryPi:RP2040
- added U3: W25Q128JVS, Package_SO:SOIC-8_5.23x5.23mm_P1.27mm, symbol Memory_Flash:W25Q128JVS
- added Y1: 12MHz, Crystal:Crystal_SMD_3225-4Pin_3.2x2.5mm, symbol Device:Crystal_GND24_Small
Connections:
- net +3.3V: now also J1.10 (Pin_10), C11.2, C12.2, C3.2, C6.2, C7.2, C8.2, C9.2, J3.1 (Pin_1), R4.1, R7.1, U2.1 (IOVDD), U2.10 (IOVDD), U2.22 (IOVDD), U2.33 (IOVDD), U2.42 (IOVDD), U2.43 (ADC_AVDD), U2.44 (VREG_IN), U2.48 (USB_VDD), U2.49 (IOVDD), U3.8 (VCC); no longer J1.1 (Pin_1)
- net GND: now also J1.1 (Pin_1), C10.1, C11.1, C12.1, C3.1, C4.1, C5.1, C6.1, C7.1, C8.1, C9.1, J2.2 (Pin_2), J3.8 (Pin_8), U2.57 (GND), U3.4 (GND); no longer J1.10 (Pin_10)
- net SWCLK: now also J1.5 (Pin_5), R5.2; no longer J1.6 (Pin_6)
- net SWDIO: now also J1.6 (Pin_6), R6.1; no longer J1.5 (Pin_5)
- net at J1.2 (Pin_2): now also J3.7 (Pin_7)
- net at J1.3 (Pin_3): now also J3.6 (Pin_6)
- net at J1.4 (Pin_4): now also J3.5 (Pin_5)
- net at J1.7 (Pin_7): now also J3.4 (Pin_4)
- net at J1.8 (Pin_8): now also J3.3 (Pin_3)
- net at J1.9 (Pin_9): now also J3.2 (Pin_2)
- net USB_N: now reaches J5.2 (D-)
- net USB_N: now also R2.1
- net USB_P: now reaches J5.3 (D+)
- net USB_P: now also R1.1
- new net: R3.1, R4.2, U2.56 (QSPI_SS), U3.1 (~{CS})
- new net: J2.1 (Pin_1), R3.2
- new net: R5.1, U2.4 (GPIO2)
- new net: C5.2, U2.21 (XOUT), Y1.3
- new net: U2.55 (QSPI_SD1), U3.2 (DO(IO1))
- new net: U2.54 (QSPI_SD2), U3.3 (IO2)
- new net: U2.53 (QSPI_SD0), U3.5 (DI(IO0))
- new net: U2.51 (QSPI_SD3), U3.7 (IO3)
- new net: D1.2 (A), R7.2
- new net: C4.2, U2.20 (XIN), Y1.1
- new net: R6.2, U2.5 (GPIO3)
- new net +1V1: C10.2, U2.23 (DVDD), U2.45 (VREG_VOUT), U2.50 (DVDD)
- new net QCLK: U2.52 (QSPI_SCLK), U3.6 (CLK)
- new net STS: D1.1 (K), U2.37 (GPIO25)
- new net USB+: R1.2, U2.47 (USB_DP)
- new net USB-: R2.2, U2.46 (USB_DM)
- no-connect marks 8 -> 31
Other:
- note added: "Place close to pin 44"
- note added: "Place close to pin 45"
- moved on the sheet: C1, C2, J1, J5, U1
